File: ControllerBoard/v2.sch (EAGLE design)
At the start: 28 parts, among them J5 U-F-M5DD-Y-L, SW1 SPST_TACT-EVQQ2, SW2 SPST_TACT-EVQQ2, SW6 SPST_TACT-EVQQ2, U1 JOYSTICKPTH, U3 JOYSTICKPTH, U4 SPX3819-3.3, U5 MCP73831T-2ACI/OT, X1 JSTPH

Commit message: Do the thing
Parts:
- removed SW1, SW2, SW6: SPST_TACT-EVQQ2, adafruit:SPST_TACT-EVQQ2
- added R10, R11, R12: 10k, adafruit:R-US_R0603
- added U$1: RPI-ZERO, RPI-Zero:RPI-ZERO
- added U$10, U$12, U$13, U$14, U$8, U$9: CHERRY-MX-LED, cherrymx:CHERRY-MX-LED
- added U2: MCP3008-I/SL, MCP3008-I_SL:MCP3008-I/SL
Connections:
- new net BTN_D: R10.1, U$12.SW1
- new net BTN_E: R11.1, U$13.SW1
- new net BTN_F: R12.1, U$14.SW1
- new net CE0: U$1.!CE0!/GPIO8, U2.!CS/SHDN
- new net MISO: U$1.GPIO9/MISO, U2.DOUT
- new net MOSI: U$1.GPIO10/MOSI, U2.DIN
- new net SCLK: U$1.GPIO11/SCLK, U2.CLK
- net 3.3V: now also R10.2, R11.2, R12.2, U2.VDD, U2.VREF
- net BTN_A: now also U$1.GPIO5, U$8.SW1; no longer SW6.S, SW6.S1
- net BTN_B: now also U$1.GPIO6, U$9.SW1; no longer SW1.S, SW1.S1
- net BTN_C: now also U$1.GPIO13, U$10.SW1; no longer SW2.S, SW2.S1
- net GND: now also U$10.SW2, U$12.SW2, U$13.SW2, U$14.SW2, U$8.SW2, U$9.SW2, U2.AGND, U2.DGND; no longer SW1.P, SW1.P1, SW2.P, SW2.P1, SW6.P, SW6.P1
- net H1: now also U2.CH1
- net H2: now also U2.CH3
- net V1: now also U2.CH0
- net V2: now also U2.CH2
Other:
- moved on the sheet: J5, ON4, R1, R2, R4, R5, R6, R7, U1, U3

Commit message: Boards ready for review
Parts:
- removed U$10, U$12, U$13, U$14, U$8, U$9: CHERRY-MX-LED, cherrymx:CHERRY-MX-LED
- removed X1: JSTPH, microbuilder:CON_JST_PH_2PIN
- added CN1: (no value), adafruit:JST_2PIN-THM-RA
- added S1, S2, S3, S4, S5, S6: B3F-4050, B3F-4050:B3F-4050
Connections:
- new net N$7: U$1.GPIO21
- net BATTERY_SENSE: now also U2.CH4
- net BTN_A: now also S1.NO; no longer U$8.SW1
- net BTN_B: now also S5.NO; no longer U$9.SW1
- net BTN_C: now also S6.NO; no longer U$10.SW1
- net BTN_D: now also S2.NO, U$1.GPIO19; no longer U$12.SW1
- net BTN_E: now also S3.NO, U$1.GPIO26; no longer U$13.SW1
- net BTN_F: now also S4.NO, U$1.GPIO20; no longer U$14.SW1
- net GND: now also CN1.1, S1.COM, S2.COM, S3.COM, S4.COM, S5.COM, S6.COM; no longer U$10.SW2, U$12.SW2, U$13.SW2, U$14.SW2, U$8.SW2, U$9.SW2, X1.1
- net N$2: now also CN1.2; no longer X1.2

Commit message: Added Breakout Board2
Parts:
- removed C14: 1uF, microbuilder:CAP_CERAMIC0603_NO
Connections:
- removed net AREF: C14.1
- removed net B_1: U3.SEL-
- removed net B_2: U1.SEL-
- net 3.3V: now also U$1.3V3@1, U$1.3V3@2; no longer U1.SEL+, U3.SEL+
- net GND: now also U$1.GND@1, U$1.GND@2, U$1.GND@3, U$1.GND@4, U$1.GND@5, U$1.GND@6, U$1.GND@7, U$1.GND@8; no longer C14.2
Changed lines of the file:
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@@
 </variantdefs>
 <classes>
-<class number="0" name="default" width="0.25" drill="0.3">
+<class number="0" name="default" width="0.15" drill="0.3">
 <clearance class="0" value="0.2"/>
 </class>
@@
 <clearance class="3" value="0.2"/>
 </class>
-<class number="4" name="5V" width="1" drill="0.3">
+<class number="4" name="5V" width="0.4" drill="0.3">
 <clearance class="4" value="0.4"/>
 </class>
@@
 <part name="U$29" library="microbuilder" deviceset="GND" device=""/>
 <part name="U$30" library="microbuilder" deviceset="GND" device=""/>
-<part name="GND12" library="supply1" deviceset="GND" device=""/>
-<part name="C14" library="microbuilder" deviceset="CAP_CERAMIC" device="0603_NO" value="1uF"/>
 <part name="+3V4" library="supply1" deviceset="+3V3" device=""/>
 <part name="U$2" library="microbuilder" deviceset="VBUS" device=""/>
@@
 <part name="S6" library="B3F-4050" deviceset="B3F-4050" device=""/>
 <part name="CN1" library="adafruit" library_urn="urn:adsk.eagle:library:420" deviceset="JST_2PIN" device="-THM-RA" package3d_urn="urn:adsk.eagle:package:6240694/1"/>
+<part name="GND16" library="supply1" deviceset="GND" device=""/>
+<part name="GND17" library="supply1" deviceset="GND" device=""/>
+<part name="U$8" library="microbuilder" deviceset="3.3V" device=""/>
 </parts>
 <sheets>
@@
 <attribute name="VALUE" x="-212.344" y="198.12" size="1.27" layer="96"/>
 </instance>
-<instance part="GND12" gate="1" x="-154.94" y="200.66" smashed="yes" rot="MR0">
-<attribute name="VALUE" x="-152.4" y="198.12" size="1.778" layer="96" rot="MR0"/>
-</instance>
-<instance part="C14" gate="G$1" x="-154.94" y="210.82" smashed="yes">
-<attribute name="NAME" x="-157.23" y="212.07" size="1.27" layer="95" font="vector" rot="R90" align="center"/>
-<attribute name="VALUE" x="-152.64" y="212.07" size="1.27" layer="96" font="vector" rot="R90" align="center"/>
-</instance>
 <instance part="+3V4" gate="G$1" x="-180.34" y="233.68" smashed="yes" rot="MR0"/>
 <instance part="U$2" gate="G$1" x="-231.14" y="233.68" smashed="yes">
@@
 <attribute name="NAME" x="-161.29" y="207.645" size="1.778" layer="95" rot="R180"/>
 <attribute name="VALUE" x="-161.29" y="218.44" size="1.778" layer="96" rot="R180"/>
+</instance>
+<instance part="GND16" gate="1" x="-254" y="17.78" smashed="yes">
+<attribute name="VALUE" x="-256.54" y="15.24" size="1.778" layer="96"/>
+</instance>
+<instance part="GND17" gate="1" x="-129.54" y="10.16" smashed="yes">
+<attribute name="VALUE" x="-132.08" y="7.62" size="1.778" layer="96"/>
+</instance>
+<instance part="U$8" gate="G$1" x="-246.38" y="96.52" smashed="yes">
+<attribute name="VALUE" x="-247.904" y="97.536" size="1.27" layer="96"/>
 </instance>
 </instances>
@@
 <pinref part="U$29" gate="G$1" pin="GND"/>
 <wire x1="-187.96" y1="205.74" x2="-187.96" y2="203.2" width="0.1524" layer="91"/>
-</segment>
-<segment>
-<pinref part="GND12" gate="1" pin="GND"/>
-<pinref part="C14" gate="G$1" pin="2"/>
-<wire x1="-154.94" y1="208.28" x2="-154.94" y2="203.2" width="0.1524" layer="91"/>
 </segment>
 <segment>
@@
 <wire x1="-45.72" y1="22.86" x2="-50.8" y2="22.86" width="0.1524" layer="91"/>
 <pinref part="GND7" gate="1" pin="GND"/>
+<junction x="-45.72" y="22.86"/>
 </segment>
 <segment>
@@
 <pinref part="GND8" gate="1" pin="GND"/>
 <wire x1="-144.78" y1="154.94" x2="-144.78" y2="149.86" width="0.1524" layer="91"/>
+</segment>
+<segment>
+<pinref part="U$1" gate="G$1" pin="GND@1"/>
+<wire x1="-210.82" y1="73.66" x2="-254" y2="73.66" width="0.1524" layer="91"/>
+<pinref part="U$1" gate="G$1" pin="GND@2"/>
+<wire x1="-210.82" y1="53.34" x2="-254" y2="53.34" width="0.1524" layer="91"/>
+<wire x1="-254" y1="53.34" x2="-254" y2="35.56" width="0.1524" layer="91"/>
+<pinref part="U$1" gate="G$1" pin="GND@3"/>
+<wire x1="-254" y1="35.56" x2="-254" y2="20.32" width="0.1524" layer="91"/>
+<wire x1="-210.82" y1="35.56" x2="-254" y2="35.56" width="0.1524" layer="91"/>
+<junction x="-254" y="35.56"/>
+<wire x1="-254" y1="73.66" x2="-254" y2="53.34" width="0.1524" layer="91"/>
+<junction x="-254" y="53.34"/>
+<pinref part="GND16" gate="1" pin="GND"/>
+</segment>
+<segment>
+<pinref part="U$1" gate="G$1" pin="GND@8"/>
+<wire x1="-162.56" y1="78.74" x2="-129.54" y2="78.74" width="0.1524" layer="91"/>
+<wire x1="-129.54" y1="78.74" x2="-129.54" y2="68.58" width="0.1524" layer="91"/>
+<pinref part="U$1" gate="G$1" pin="GND@7"/>
+<wire x1="-129.54" y1="68.58" x2="-129.54" y2="60.96" width="0.1524" layer="91"/>
+<wire x1="-129.54" y1="60.96" x2="-129.54" y2="48.26" width="0.1524" layer="91"/>
+<wire x1="-129.54" y1="48.26" x2="-129.54" y2="43.18" width="0.1524" layer="91"/>
+<wire x1="-129.54" y1="43.18" x2="-129.54" y2="12.7" width="0.1524" layer="91"/>
+<wire x1="-162.56" y1="43.18" x2="-129.54" y2="43.18" width="0.1524" layer="91"/>
+<junction x="-129.54" y="43.18"/>
+<pinref part="U$1" gate="G$1" pin="GND@6"/>
+<wire x1="-162.56" y1="48.26" x2="-129.54" y2="48.26" width="0.1524" layer="91"/>
+<junction x="-129.54" y="48.26"/>
+<pinref part="U$1" gate="G$1" pin="GND@5"/>
+<wire x1="-162.56" y1="60.96" x2="-129.54" y2="60.96" width="0.1524" layer="91"/>
+<junction x="-129.54" y="60.96"/>
+<pinref part="U$1" gate="G$1" pin="GND@4"/>
+<wire x1="-162.56" y1="68.58" x2="-129.54" y2="68.58" width="0.1524" layer="91"/>
+<junction x="-129.54" y="68.58"/>
+<pinref part="GND17" gate="1" pin="GND"/>
 </segment>
 </net>
@@
 </segment>
 <segment>
-<pinref part="U1" gate="G$1" pin="SEL+"/>
-<wire x1="86.36" y1="172.72" x2="78.74" y2="172.72" width="0.1524" layer="91"/>
-<label x="78.74" y="172.72" size="1.778" layer="95"/>
-</segment>
-<segment>
-<pinref part="U3" gate="G$1" pin="SEL+"/>
-<wire x1="86.36" y1="213.36" x2="78.74" y2="213.36" width="0.1524" layer="91"/>
-<label x="78.74" y="213.36" size="1.778" layer="95"/>
-</segment>
-<segment>
 <pinref part="U2" gate="A" pin="VDD"/>
 <wire x1="-50.8" y1="66.04" x2="-45.72" y2="66.04" width="0.1524" layer="91"/>
@@
 <wire x1="-144.78" y1="132.08" x2="-144.78" y2="134.62" width="0.1524" layer="91"/>
 <label x="-152.4" y="134.62" size="1.778" layer="95"/>
+</segment>
+<segment>
+<pinref part="U$8" gate="G$1" pin="3.3V"/>
+<pinref part="U$1" gate="G$1" pin="3V3@1"/>
+<wire x1="-246.38" y1="93.98" x2="-246.38" y2="83.82" width="0.1524" layer="91"/>
+<wire x1="-246.38" y1="83.82" x2="-228.6" y2="83.82" width="0.1524" layer="91"/>
+<pinref part="U$1" gate="G$1" pin="3V3@2"/>
+<wire x1="-228.6" y1="83.82" x2="-210.82" y2="83.82" width="0.1524" layer="91"/>
+<wire x1="-210.82" y1="63.5" x2="-228.6" y2="63.5" width="0.1524" layer="91"/>
+<wire x1="-228.6" y1="63.5" x2="-228.6" y2="83.82" width="0.1524" layer="91"/>
+<junction x="-228.6" y="83.82"/>
 </segment>
 </net>
@@
 <pinref part="U$1" gate="G$1" pin="GPIO13"/>
 <wire x1="-238.76" y1="43.18" x2="-210.82" y2="43.18" width="0.1524" layer="91"/>
-</segment>
-</net>
-<net name="AREF" class="0">
-<segment>
-<pinref part="C14" gate="G$1" pin="1"/>
-<wire x1="-154.94" y1="215.9" x2="-154.94" y2="226.06" width="0.1524" layer="91"/>
-<label x="-154.94" y="218.44" size="1.778" layer="95" rot="R90"/>
 </segment>
 </net>
@@
 </segment>
 </net>
-<net name="B_1" class="0">
-<segment>
-<pinref part="U3" gate="G$1" pin="SEL-"/>
-<wire x1="86.36" y1="210.82" x2="83.82" y2="210.82" width="0.1524" layer="91"/>
-<label x="81.28" y="210.82" size="1.778" layer="95"/>
-</segment>
-</net>
-<net name="B_2" class="0">
-<segment>
-<pinref part="U1" gate="G$1" pin="SEL-"/>
-<wire x1="86.36" y1="170.18" x2="83.82" y2="170.18" width="0.1524" layer="91"/>
-<label x="78.74" y="170.18" size="1.778" layer="95"/>
-</segment>
-</net>
 <net name="N$2" class="0">
 <segment>
@@
 </sheet>
 </sheets>
+<errors>
+</errors>
 </schematic>
 </drawing>
